File: cats/cat_pcb_2/cat_pcb_2.kicad_pcb (KiCad board)
At the start: 2 copper layers, 43.5 x 64 mm, 6 parts, among them SW1 SMT_SPDT

Commit message: Bunch of changes
Other:
- board text added: "+ POSITIVE +"
