File: ghosts/ghost_pcb_2/ghost_pcb_2.kicad_pcb (KiCad board)
At the start: 2 copper layers, 67.4 x 83.5 mm, 6 parts, among them SW1 SMT_SPDT

Commit message: Bunch of changes
Parts:
- D1, D2: moved to B.Cu
- moved D2 0.07 mm to (130.8, 80.8)
